File: judo-devkit/judo-devkit_v1.brd (EAGLE design)
At the start: 71 x 32 mm, 89 parts, among them J10 USB Female Type C Connector, J11 CORTEX_DEBUG, J3 QWIIC_RIGHT_ANGLE, U1 LTC4411ES5TRMPBF, U2 3.3V, U4 ARTEMIS_MODULESMD, U5 BME280, U6 CH340E_MSOP10, Y2 32.768kHz

Commit message: routing
Parts:
- moved C18 73.5 mm to (33.9, 2.31)
- moved C17 63.1 mm to (33.7, 4.31)
- moved C4 54.1 mm to (39.3, 2.31)
- moved TP8 47.9 mm to (51.0, 4.00)
- moved R2 43.8 mm to (51.0, 2.00)
- moved CFIL1 43.1 mm to (54.0, 27.0), turned to 180 degrees
- moved C28 40.5 mm to (16.0, 19.0), turned to 180 degrees
- moved C6 40.4 mm to (48.0, 26.0)
- moved U1 34.6 mm to (44.0, 5.00)
- moved R9 34.4 mm to (48.0, 4.00)
- moved C1 30.9 mm to (46.0, 9.00), flipped to the bottom, turned to 270 degrees
- moved RSET2 29.6 mm to (59.9, 10.2), turned to 0 degrees
- moved U$1 26.6 mm to (43.1, 10.2), turned to 0 degrees
- moved TDBIAS_VCC 23.2 mm to (57.0, 22.0)
- moved REGULATOR1 20.5 mm to (54.0, 22.0), turned to 180 degrees
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Routing:
- net VDD: track 0.00 -> 77.2 mm
- net GND: track 0.00 -> 48.5 mm, vias 0 -> 3
- net !RTS: track 0.00 -> 44.0 mm, vias 0 -> 1
- net !RESET: track 0.00 -> 42.1 mm
- net PDMDATA: track 0.00 -> 41.1 mm
- net V_USB: track 0.00 -> 37.3 mm
- net ~A1: track 0.00 -> 30.6 mm
- net VCC: track 0.00 -> 28.9 mm, vias 0 -> 2
- net VIN: track 0.00 -> 27.1 mm, vias 0 -> 1
- net ~D27/SCL2: track 0.00 -> 26.7 mm, vias 0 -> 2
- net SWDCK: track 0.00 -> 24.4 mm, vias 0 -> 1
- net SWDIO: track 0.00 -> 23.6 mm, vias 0 -> 1
- net PDMCLK: track 0.00 -> 23.3 mm
- net ~D25/SDA2: track 0.00 -> 22.0 mm, vias 0 -> 2
- net TDBIAS: track 0.00 -> 20.1 mm
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Other:
- board size 71 x 32 mm -> 72 x 32 mm

Commit message: more routing, it looks pretty messy sadly
Parts:
- moved R19 39.7 mm to (5.00, 23.0), flipped to the bottom
- moved R11 22.2 mm to (8.00, 20.0), flipped to the bottom, turned to 0 degrees
- moved C22 18.0 mm to (32.0, 8.00)
- moved C19 18.0 mm to (34.0, 8.00)
- moved C23 18.0 mm to (37.0, 8.00)
- moved R12 17.1 mm to (9.00, 23.0), flipped to the bottom, turned to 0 degrees
- moved Y2 15.8 mm to (1.85, 17.4), flipped to the bottom, turned to 270 degrees
- moved R3 12.6 mm to (29.0, 11.0), flipped to the bottom, turned to 0 degrees
- moved R15 10.8 mm to (29.0, 18.0)
- moved R7 10.8 mm to (31.0, 18.0)
- moved R16 9.00 mm to (33.0, 18.0)
- moved R10 8.07 mm to (29.0, 13.0), flipped to the bottom, turned to 0 degrees
- moved R1 3.16 mm to (22.0, 19.0)
- moved C17 1.41 mm to (34.7, 5.31)
- moved TP4 1.41 mm to (9.00, 16.0)
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Routing:
- net ~MOSI: track 0.00 -> 32.6 mm, vias 0 -> 1
- net N$4: track 0.00 -> 30.9 mm, vias 0 -> 3
- net ~MISO: track 0.00 -> 24.4 mm, vias 0 -> 1
- net ~A1: track 30.6 -> 53.5 mm, vias 0 -> 1
- net TXO-0_R: track 0.00 -> 20.1 mm, vias 0 -> 1
- net ~A0: track 0.00 -> 20.0 mm, vias 0 -> 1
- net ~SCK: track 0.00 -> 17.4 mm, vias 0 -> 2
- net N$14: track 0.00 -> 15.6 mm, vias 0 -> 2
- net ~TXO-0: track 0.00 -> 12.2 mm, vias 0 -> 1
- net N$8: track 0.00 -> 11.7 mm, vias 0 -> 1
- net BOOT: track 3.91 -> 15.5 mm, vias 0 -> 1
- net ~A2: track 0.00 -> 11.5 mm, vias 0 -> 1
- net N$7: track 0.00 -> 11.2 mm, vias 0 -> 1
- net N$6: track 0.00 -> 11.1 mm, vias 0 -> 1
- net N$15: track 0.00 -> 10.1 mm, vias 0 -> 1
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